File: eagle/fab_scope.brd (EAGLE design)
At the start: 39 parts, among them IC1 ULN2003AN, K1 FRS1B, K2 FRS1B, K3 FRS1B, K4 FRS1B, K5 FRS1B, K6 FRS1B

Commit message: added new board and imgs
Parts:
- removed BUTTONS_1: (no value), con-lstb:MA03-1
- removed K3, K4, K5, K6: FRS1B, relay:FRS1B
- removed LEDS: (no value), con-amp-quick:02P
- removed R1, R4, R5, RB3: 10k, fab:R1206
- removed R7, R8: 499k, fab:R1206
- added BUTTON_F, BUTTON_V: M01PTH_LONGPAD, 01_SparkFun:1X01_LONGPAD
- moved R9 74.3 mm to (46.7, 10.7), turned to 270 degrees
- moved PROBES_VCC 70.7 mm to (40.1, 9.65), turned to 0 degrees
- moved R6 44.3 mm to (33.3, 9.91)
- moved RB1 35.7 mm to (22.9, 34.3), turned to 90 degrees
- moved K2 22.7 mm to (30.7, 19.1)
- moved K1 12.5 mm to (41.4, 19.6), turned to 0 degrees
- moved IC1 2.74 mm to (35.1, 33.3)
- moved RB2 2.54 mm to (29.7, 68.8)
Connections:
- removed net BUTTON_S: 1284P.42, BUTTONS_1.3, RB2.2
- removed net N$10: K1.O, K2.P@
- removed net N$12: K4.O, K5.P@
- removed net N$13: K5.O, K6.P@
- removed net N$15: 1284P.35, LEDS.2
- removed net N$16: 1284P.34, LEDS.1
- removed net N$17: R1.2, R4.1
- removed net N$27: IC1.10, K1.2
- removed net N$28: IC1.11, K2.2
- removed net N$29: IC1.12, K3.2
- removed net N$30: IC1.13, K4.2
- removed net N$31: IC1.14, K5.2
- removed net N$32: IC1.15, K6.2
- removed net N$33: IC1.16
- removed net N$7: K4.S, R7.1
- removed net N$8: K5.S, R8.1
- removed net N$9: K2.S, R5.1
- removed net RELAY_3: 1284P.20, IC1.3
- removed net RELAY_4: 1284P.19, IC1.4
- removed net RELAY_5: 1284P.16, IC1.5
- removed net RELAY_6: 1284P.15, IC1.6
- removed net RELAY_7: 1284P.14, IC1.7
- net BUTTON_F: now also 1284P.11, BUTTON_F.1; no longer 1284P.41, BUTTONS_1.2
- net BUTTON_V: now also 1284P.42, BUTTON_V.1, RB2.2; no longer 1284P.40, BUTTONS_1.1, RB3.1
- net GND: now also K2.P@; no longer K1.P@, RB3.2
- net N$11: now also K2.S; no longer K3.S
- net N$14: now also K1.S; no longer K6.S
- net N$4: now also IC1.10, K2.2; no longer K2.O, K3.P@
- net N$5: now also IC1.13, K1.2; no longer K1.S, R1.1
- net PROBE: now also K1.P@; no longer K4.P, R4.2, R5.2
- net RELAY_1: now also 1284P.21, IC1.4; no longer 1284P.22, IC1.1
- net RELAY_2: now also 1284P.16, IC1.7; no longer 1284P.21, IC1.2
- net VCC: no longer K3.1, K4.1, K5.1, K6.1
- net V_PROBES: now also K1.O; no longer K6.O, R7.2, R8.2
Routing:
- net VCC: track 402.7 -> 156.4 mm
- net N$32: track 69.4 -> 0.00 mm
- net PROBE: track 227.5 -> 165.5 mm
- net V_PROBES: track 70.6 -> 14.1 mm
- net N$31: track 53.9 -> 0.00 mm
- net N$29: track 46.1 -> 0.00 mm
- net N$30: track 38.5 -> 0.00 mm
- net N$28: track 26.6 -> 0.00 mm
- net N$16: track 19.3 -> 0.00 mm
- net N$15: track 17.4 -> 0.00 mm
- net BUTTON_S: track 13.7 -> 0.00 mm
- net N$24: track 126.8 -> 114.2 mm
- net RELAY_3: track 11.0 -> 0.00 mm
- net N$10: track 10.7 -> 0.00 mm
- net N$14: track 3.91 -> 14.5 mm
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Other:
- board text added: "Fab"
- board text added: "Scope"
