File: eagle/fab_scope.sch (EAGLE design)
At the start: 39 parts, among them IC1 ULN2003AN, K1 FRS1B, K2 FRS1B, K3 FRS1B, K4 FRS1B, K5 FRS1B, K6 FRS1B

Commit message: added new board and imgs
Parts:
- removed BUTTONS_1: (no value), con-lstb:MA03-1
- removed K3, K4, K5, K6: FRS1B, relay:FRS1B
- removed LEDS: (no value), con-amp-quick:M02
- removed R1, R4, R5, RB3: 10k, fab:RES-US1206
- removed R7, R8: 499k, fab:RES-US1206
- added BUTTON_F, BUTTON_V: M01PTH_LONGPAD, 01_SparkFun:M01PTH_LONGPAD
Connections:
- removed net BUTTON_S: 1284P.PB2, BUTTONS_1.3, RB2.2
- removed net N$10: K12.O, K22.P@1
- removed net N$12: K42.O, K52.P@1
- removed net N$13: K52.O, K62.P@1
- removed net N$15: 1284P.PA2, LEDS.2
- removed net N$16: 1284P.PA3, LEDS.1
- removed net N$17: R1.2, R4.1
- removed net N$27: IC1.O7, K11.2
- removed net N$28: IC1.O6, K21.2
- removed net N$29: IC1.O5, K31.2
- removed net N$30: IC1.O4, K41.2
- removed net N$31: IC1.O3, K51.2
- removed net N$32: IC1.O2, K61.2
- removed net N$33: IC1.O1
- removed net N$7: K42.S, R7.1
- removed net N$8: K52.S, R8.1
- removed net N$9: K22.S, R5.1
- removed net RELAY_3: 1284P.PC1, IC1.I3
- removed net RELAY_4: 1284P.PC0, IC1.I4
- removed net RELAY_5: 1284P.PD7, IC1.I5
- removed net RELAY_6: 1284P.PD6, IC1.I6
- removed net RELAY_7: 1284P.PD5, IC1.I7
- net BUTTON_F: now also 1284P.PD2, BUTTON_F.1; no longer 1284P.PB1, BUTTONS_1.2
- net BUTTON_V: now also 1284P.PB2, BUTTON_V.1, RB2.2; no longer 1284P.PB0, BUTTONS_1.1, RB3.1
- net GND: now also K22.P@1; no longer K12.P@1, RB3.2
- net N$11: now also K22.S; no longer K32.S
- net N$14: now also K12.S; no longer K62.S
- net N$4: now also IC1.O7, K21.2; no longer K22.O, K32.P@1
- net N$5: now also IC1.O4, K11.2; no longer K12.S, R1.1
- net PROBE: now also K12.P@1; no longer K42.P, R4.2, R5.2
- net RELAY_1: now also 1284P.PC2, IC1.I4; no longer 1284P.PC3, IC1.I1
- net RELAY_2: now also 1284P.PD7, IC1.I7; no longer 1284P.PC2, IC1.I2
- net VCC: no longer K31.1, K41.1, K51.1, K61.1
- net V_PROBES: now also K12.O; no longer K62.O, R7.2, R8.2
Other:
- moved on the sheet: K1, K2, R6, R9, RB1, RB2
